File: kicad/Motherboard/Motherboard.kicad_sch (KiCad schematic)
At the start: 52 parts, among them J1 Conn_01x16_Pin, J1 USB_C_Receptacle_USB2.0, J2 Conn_01x16_Pin, J3 Conn_01x16_Pin, J4 Conn_01x16_Pin, J5 Conn_01x02_Pin, J6 Conn_01x04_Pin, J7 Conn_01x04_Pin, Q1 DMN3404L, SW1 Reset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

Commit message: updated schematic
Parts:
- C1, C3, C4, C5: footprint (none) -> Capacitor_SMD:C_0402_1005Metric_Pad0.74x0.62mm_HandSolder
- C2: footprint (none) -> Capacitor_SMD:C_0603_1608Metric_Pad1.08x0.95mm_HandSolder
- C6: footprint (none) -> Capacitor_SMD:C_0805_2012Metric_Pad1.18x1.45mm_HandSolder
- C7: footprint (none) -> Capacitor_SMD:C_1206_3216Metric_Pad1.33x1.80mm_HandSolder
- C8: footprint (none) -> Capacitor_SMD:C_1210_3225Metric_Pad1.33x2.70mm_HandSolder
- J1, SW1, SW2: footprint (none) -> Button_Switch_SMD:SW_Push_SPST_NO_Alps_SKRK
- R1, R2, R3, R4, R5: footprint (none) -> Resistor_SMD:R_0402_1005Metric_Pad0.72x0.64mm_HandSolder
- renumbered J1 to J8
Connections:
- net +5V: now also D2.1 (K); no longer D2.2 (A)
- net GND: now also D1.2 (A); no longer D1.1 (K)
- net at J5.1 (Pin_1), Q1.3 (D): now also D2.2 (A); no longer D2.1 (K)
- net at L1.1, U9.2 (OUT): now also D1.1 (K); no longer D1.2 (A)
Other:
- moved on the sheet: D1, D2
Changed lines of the file:
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@@
 	)
 	(junction
+		(at 77.47 187.96)
+		(diameter 0)
+		(color 0 0 0 0)
+	)
+	(junction
 		(at 241.3 24.13)
 		(diameter 0)
@@
 	)
 	(junction
-		(at 77.47 187.96)
-		(diameter 0)
-		(color 0 0 0 0)
-	)
-	(junction
 		(at 115.57 142.24)
 		(diameter 0)
@@
 	(wire
 		(pts
-			(xy 228.6 123.19) (xy 226.06 123.19)
-		)
-		(stroke
-			(width 0)
-			(type default)
-		)
-	)
-	(wire
-		(pts
 			(xy 228.6 31.75) (xy 241.3 31.75)
 		)
@@
 	(wire
 		(pts
-			(xy 77.47 187.96) (xy 93.98 187.96)
-		)
-		(stroke
-			(width 0)
-			(type default)
-		)
-	)
-	(wire
-		(pts
 			(xy 144.78 176.53) (xy 142.24 176.53)
 		)
@@
 	(wire
 		(pts
+			(xy 77.47 187.96) (xy 93.98 187.96)
+		)
+		(stroke
+			(width 0)
+			(type default)
+		)
+	)
+	(wire
+		(pts
 			(xy 248.92 162.56) (xy 254 162.56)
 		)
@@
 	(wire
 		(pts
-			(xy 77.47 180.34) (xy 82.55 180.34)
+			(xy 60.96 187.96) (xy 77.47 187.96)
 		)
 		(stroke
@@
 	(wire
 		(pts
-			(xy 60.96 187.96) (xy 77.47 187.96)
+			(xy 77.47 180.34) (xy 82.55 180.34)
 		)
 		(stroke
@@
 		(dnp no)
 		(property "Reference" "J2"
-			(at 179.324 57.15 90)
+			(at 178.816 59.436 90)
 			(effects
 				(font
@@
 		(on_board yes)
 		(dnp no)
-		(property "Reference" "J1"
-			(at 137.16 56.388 90)
+		(property "Reference" "J8"
+			(at 136.906 58.42 90)
 			(effects
 				(font
@@
 			(project ""
 				(path "/6e7606c8-26d5-4d26-b509-210c4758a44d"
-					(reference "J1")
+					(reference "J8")
 					(unit 1)
 				)
@@
 	(symbol
 		(lib_id "Device:D_Schottky")
-		(at 123.19 180.34 180)
+		(at 123.19 180.34 0)
 		(unit 1)
 		(exclude_from_sim no)
@@
 		(dnp no)
 		(property "Reference" "D2"
-			(at 128.27 181.61 90)
+			(at 118.11 179.07 90)
 			(effects
 				(font
@@
 		)
 		(property "Value" "1N5819"
-			(at 119.38 183.134 0)
+			(at 126.492 183.388 0)
 			(effects
 				(font
@@
 			)
 		)
-		(property "Footprint" ""
+		(property "Footprint" "Capacitor_SMD:C_0603_1608Metric_Pad1.08x0.95mm_HandSolder"
 			(at 229.5652 31.75 0)
 			(effects
@@
 			)
 		)
-		(property "Footprint" ""
+		(property "Footprint" "Resistor_SMD:R_0402_1005Metric_Pad0.72x0.64mm_HandSolder"
 			(at 138.43 189.992 90)
 			(effects
@@
 			)
 		)
-		(property "Footprint" ""
+		(property "Footprint" "Capacitor_SMD:C_0402_1005Metric_Pad0.74x0.62mm_HandSolder"
 			(at 192.7352 27.94 0)
 			(effects
@@
 			)
 		)
-		(property "Footprint" ""
+		(property "Footprint" "Capacitor_SMD:C_0402_1005Metric_Pad0.74x0.62mm_HandSolder"
 			(at 261.62 21.2852 0)
 			(effects
@@
 			)
 		)
-		(property "Footprint" ""
+		(property "Footprint" "Capacitor_SMD:C_1206_3216Metric_Pad1.33x1.80mm_HandSolder"
 			(at 37.7952 185.42 0)
 			(effects
@@
 			)
 		)
-		(property "Footprint" ""
+		(property "Footprint" "Capacitor_SMD:C_1210_3225Metric_Pad1.33x2.70mm_HandSolder"
 			(at 94.9452 187.96 0)
 			(effects
@@
 			)
 		)
-		(property "Footprint" ""
+		(property "Footprint" "Resistor_SMD:R_0402_1005Metric_Pad0.72x0.64mm_HandSolder"
 			(at 136.398 187.96 90)
 			(effects
@@
 			)
 		)
-		(property "Footprint" ""
+		(property "Footprint" "Button_Switch_SMD:SW_Push_SPST_NO_Alps_SKRK"
 			(at 265.43 35.56 0)
 			(effects
@@
 			)
 		)
-		(property "Footprint" ""
+		(property "Footprint" "Capacitor_SMD:C_0402_1005Metric_Pad0.74x0.62mm_HandSolder"
 			(at 187.6552 147.32 0)
 			(effects
@@
 	(symbol
 		(lib_id "power:GND")
-		(at 226.06 123.19 0)
+		(at 228.6 123.19 0)
 		(unit 1)
 		(exclude_from_sim no)
@@
 		(dnp no)
 		(property "Reference" "#PWR07"
-			(at 226.06 129.54 0)
+			(at 228.6 129.54 0)
 			(effects
 				(font
@@
 		)
 		(property "Value" "GND"
-			(at 229.362 122.936 0)
+			(at 231.902 122.936 0)
 			(effects
 				(font
@@
 		)
 		(property "Footprint" ""
-			(at 226.06 123.19 0)
+			(at 228.6 123.19 0)
 			(effects
 				(font
@@
 		)
 		(property "Datasheet" ""
-			(at 226.06 123.19 0)
+			(at 228.6 123.19 0)
 			(effects
 				(font
@@
 		)
 		(property "Description" ""
-			(at 226.06 123.19 0)
+			(at 228.6 123.19 0)
 			(effects
 				(font
@@
 			)
 		)
-		(property "Footprint" ""
+		(property "Footprint" "Resistor_SMD:R_0402_1005Metric_Pad0.72x0.64mm_HandSolder"
 			(at 255.778 158.75 90)
 			(effects
@@
 			)
 		)
-		(property "Footprint" ""
+		(property "Footprint" "Resistor_SMD:R_0402_1005Metric_Pad0.72x0.64mm_HandSolder"
 			(at 207.01 31.242 90)
 			(effects
@@
 	(symbol
 		(lib_id "Device:D_Schottky")
-		(at 77.47 184.15 90)
+		(at 77.47 184.15 270)
 		(unit 1)
 		(exclude_from_sim no)
@@
 		(dnp no)
 		(property "Reference" "D1"
-			(at 74.422 181.356 90)
+			(at 80.518 186.944 90)
 			(effects
 				(font
@@
 		)
 		(property "Value" "1N5819"
-			(at 80.264 180.086 0)
+			(at 74.676 188.214 0)
 			(effects
 				(font
@@
 			)
 		)
-		(property "Footprint" ""
+		(property "Footprint" "Button_Switch_SMD:SW_Push_SPST_NO_Alps_SKRK"
 			(at 205.74 24.13 0)
 			(effects
@@
 			)
 		)
-		(property "Footprint" ""
+		(property "Footprint" "Capacitor_SMD:C_0402_1005Metric_Pad0.74x0.62mm_HandSolder"
 			(at 242.2652 31.75 0)
 			(effects
@@
 			)
 		)
-		(property "Footprint" ""
+		(property "Footprint" "Resistor_SMD:R_0402_1005Metric_Pad0.72x0.64mm_HandSolder"
 			(at 259.842 158.75 90)
 			(effects
@@
 			)
 		)
-		(property "Footprint" ""
+		(property "Footprint" "Capacitor_SMD:C_0805_2012Metric_Pad1.18x1.45mm_HandSolder"
 			(at 220.6752 147.32 0)
 			(effects
@@
 			)
 		)
-		(property "Footprint" ""
+		(property "Footprint" "Button_Switch_SMD:SW_Push_SPST_NO_Alps_SKRK"
 			(at 251.46 140.97 0)
 			(effects

Commit message: tmcs done
Parts:
- R6, R7, R8, R9: value R -> .1
Connections:
- net +5V: no longer U7.22 (VS), U7.28 (VS), U8.22 (VS), U8.28 (VS)
- net MS2_A: now reaches U7.10 (MS2)
- net Diag_A: now reaches U7.11 (DIAG)
- net Index_A: now reaches U7.12 (INDEX)
- net VCC3V3: now reaches U7.15 (VCC_IO)
- net VCC3V3: now also U8.15 (VCC_IO)
- net Step_A: now reaches U7.16 (STEP)
- net Dir_A: now reaches U7.19 (DIR)
- net ENN_A: now reaches U7.2 (ENN)
- net MS1_A: now reaches U7.9 (MS1)
- net MS2_B: now reaches U8.10 (MS2)
- net Diag_B: now reaches U8.11 (DIAG)
- net Index_B: now reaches U8.12 (INDEX)
- net Step_B: now reaches U8.16 (STEP)
- net Dir_B: now reaches U8.19 (DIR)
- net ENN_B: now reaches U8.2 (ENN)
- net MS1_B: now reaches U8.9 (MS1)
- new net M1_DC_12V: U7.22 (VS), U7.28 (VS)
- new net M2_DC_12V: U8.22 (VS), U8.28 (VS)
- no-connect marks 29 -> 21
Other:
- moved on the sheet: C15, C16, C17, C18, R10, R11, R6, R7, R8, R9, U7, U8

Commit message: penultimate schematic
Parts:
- removed R10, R11: 10R, symbol Device:R
- added C19: 2.2uF, Capacitor_SMD:C_0603_1608Metric_Pad1.08x0.95mm_HandSolder, symbol Device:C
- added C20, C21, C22, C23, C24: 22uF, Capacitor_SMD:C_0805_2012Metric_Pad1.18x1.45mm_HandSolder, symbol Device:C
- C10, C13, C9: value 100nF -> 22uF; footprint (none) -> Capacitor_SMD:C_0805_2012Metric_Pad1.18x1.45mm_HandSolder
- C11, C14: value 100uF -> 22uF; footprint (none) -> Capacitor_SMD:C_0805_2012Metric_Pad1.18x1.45mm_HandSolder
- C12: footprint (none) -> Capacitor_SMD:C_0402_1005Metric_Pad0.74x0.62mm_HandSolder
- C15: value 100nF -> 2.2uF; footprint (none) -> Capacitor_SMD:C_0603_1608Metric_Pad1.08x0.95mm_HandSolder
- C16: value 100nF -> 22nF; footprint (none) -> Capacitor_SMD:C_0201_0603Metric_Pad0.64x0.40mm_HandSolder
- C17: footprint (none) -> Capacitor_SMD:C_0201_0603Metric_Pad0.64x0.40mm_HandSolder
- C18: value 22nF -> 100nF; footprint (none) -> Capacitor_SMD:C_0402_1005Metric_Pad0.74x0.62mm_HandSolder
- D1, D2: footprint (none) -> Diode_THT:D_DO-41_SOD81_P5.08mm_Vertical_AnodeUp
- J2, J3, J4, J8: footprint (none) -> Connector_PinHeader_1.27mm:PinHeader_1x16_P1.27mm_Horizontal
- J5: footprint (none) -> Connector_PinHeader_1.27mm:PinHeader_1x02_P1.27mm_Horizontal
- J6, J7: footprint (none) -> Connector_PinHeader_1.27mm:PinHeader_1x04_P1.27mm_Horizontal
- L1: footprint (none) -> Inductor_SMD:L_1008_2520Metric_Pad1.43x2.20mm_HandSolder
- R6, R7, R8, R9: footprint (none) -> Resistor_SMD:R_0805_2012Metric_Pad1.20x1.40mm_HandSolder
- U1: footprint PCM_Espressif:ESP32-S2-SOLO -> RF_Module:ESP32-S2-MINI-1
Connections:
- net Dir_A is gone; now on net DIR_2: U7.19 (DIR)
- net Dir_B is gone; now on net DIR_1: U8.19 (DIR)
- net ENN_A is gone; now on net ENN_2: U7.2 (ENN)
- net ENN_B is gone; now on net ENN_1: U8.2 (ENN)
- net M1_DC_12V is gone; now on net +12V: U7.22 (VS), U7.28 (VS)
- net M2_DC_12V is gone; now on net +12V: U8.22 (VS), U8.28 (VS)
- net MUR_1 is gone; now on net UART_2: U7.14 (PDN_UART)
- net MUR_2 is gone; now on net UART_1: U8.14 (PDN_UART)
- net Step_A is gone; now on net STEP_2: U7.16 (STEP)
- net Step_B is gone; now on net STEP_1: U8.16 (STEP)
- net VCC3V3 is gone; now on net +3.3V: U7.15 (VCC_IO), U8.15 (VCC_IO)
- net +12V: now also C10.1, C11.1, C12.1, C13.2, C14.2, C18.1, C9.1, C20.1, C21.2, C22.1, C23.2, C24.1
- net +5V: no longer C10.1, C11.1, C12.1, C13.1, C14.1, C15.2, C16.2, C9.1
- net GND: now also C13.1, C14.1, C15.1, C19.1, C20.2, C21.1, C22.2, C23.1, C24.2; no longer C12.2, C13.2, C14.2
- net MAGCT: now also U1.29 (SPIIO7/GPIO36/FSPICLK); no longer U1.26 (GPIO45)
- net at C16.1: now also U7.4 (CPO); no longer U7.6 (VCP)
- net at U7.5 (CPI): now also C16.2; no longer C18.2
- net 5VOUT_2: now reaches U7.8 (5VOUT)
- net 5VOUT_2: now also C19.2
- net STEP_1: now reaches U1.10 (GPIO17/U1TXD/ADC2_CH6/DAC_1)
- net UART_1: now reaches U1.11 (GPIO18/U1RXD/ADC2_CH7/DAC_2/CLK_OUT3)
- net ENN_1: now reaches U1.21 (GPIO13/TOUCH13/ADC2_CH2/FSPIQ/FSPIIO7)
- net DIR_1: now reaches U1.22 (GPIO14/TOUCH14/ADC2_CH3/FSPIWP/FSPIDQS)
- net ENN_2: now reaches U1.23 (GPIO21)
- net DIR_2: now reaches U1.24 (SPIIO4/GPIO33/FSPIHD)
- net STEP_2: now reaches U1.25 (SPIIO5/GPIO34/FSPICS0)
- net UART_2: now reaches U1.28 (SPIIO6/GPIO35/FSPID)
- net VCP_1: now reaches U8.6 (VCP)
- net VCP_1: now also C12.2; no longer C15.1
- net 5VOUT_1: now reaches U8.8 (5VOUT)
- net 5VOUT_1: now also C15.2
- net Diag_A: no longer names the net of U7.11 (DIAG)
- net Diag_B: no longer names the net of U8.11 (DIAG)
- net Index_A: no longer names the net of U7.12 (INDEX)
- net Index_B: no longer names the net of U8.12 (INDEX)
- net MS1_A: no longer names the net of U7.9 (MS1)
- net MS1_B: no longer names the net of U8.9 (MS1)
- net MS2_A: no longer names the net of U7.10 (MS2)
- net MS2_B: no longer names the net of U8.10 (MS2)
- net SM_1A+ renamed Motor1_2
- net SM_1A- renamed Motor2_2
- net SM_1B+ renamed Motor3_2
- net SM_1B- renamed Motor4_2
- net SM_2A+ renamed Motor1_1
- net SM_2A- renamed Motor2_1
- net SM_2B+ renamed Motor3_1
- net SM_2B- renamed Motor4_1
- new net VCP_2: C18.2, U7.6 (VCP)
- no-connect marks 21 -> 28
Other:
- moved on the sheet: C10, C11, C17, C3, C6, C7, C8, C9, D1, D2, J5, J6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

Commit message: updated layout
Parts:
- C1, C12, C18, C3, C4, C5: footprint Capacitor_SMD:C_0402_1005Metric_Pad0.74x0.62mm_HandSolder -> Capacitor_SMD:C_0805_2012Metric_Pad1.18x1.45mm_HandSolder
- C15, C19, C2: footprint Capacitor_SMD:C_0603_1608Metric_Pad1.08x0.95mm_HandSolder -> Capacitor_SMD:C_0805_2012Metric_Pad1.18x1.45mm_HandSolder
- C16, C17: footprint Capacitor_SMD:C_0201_0603Metric_Pad0.64x0.40mm_HandSolder -> Capacitor_SMD:C_0805_2012Metric_Pad1.18x1.45mm_HandSolder
- C7: footprint Capacitor_SMD:C_1206_3216Metric_Pad1.33x1.80mm_HandSolder -> Capacitor_SMD:C_0805_2012Metric_Pad1.18x1.45mm_HandSolder
- J1: footprint Button_Switch_SMD:SW_Push_SPST_NO_Alps_SKRK -> Connector_USB:USB_C_Receptacle_HRO_TYPE-C-31-M-12
- R1, R2, R3, R4, R5: footprint Resistor_SMD:R_0402_1005Metric_Pad0.72x0.64mm_HandSolder -> Resistor_SMD:R_0805_2012Metric_Pad1.20x1.40mm_HandSolder
- U1: footprint RF_Module:ESP32-S2-MINI-1 -> Espressif:ESP32-S2-SOLO
Changed lines of the file:
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@@
 			)
 		)
-		(property "Footprint" "Capacitor_SMD:C_0201_0603Metric_Pad0.64x0.40mm_HandSolder"
+		(property "Footprint" "Capacitor_SMD:C_0805_2012Metric_Pad1.18x1.45mm_HandSolder"
 			(at 36.5252 101.6 0)
 			(effects
@@
 			)
 		)
-		(property "Footprint" "Capacitor_SMD:C_0603_1608Metric_Pad1.08x0.95mm_HandSolder"
+		(property "Footprint" "Capacitor_SMD:C_0805_2012Metric_Pad1.18x1.45mm_HandSolder"
 			(at 229.5652 31.75 0)
 			(effects
@@
 			)
 		)
-		(property "Footprint" "Resistor_SMD:R_0402_1005Metric_Pad0.72x0.64mm_HandSolder"
+		(property "Footprint" "Resistor_SMD:R_0805_2012Metric_Pad1.20x1.40mm_HandSolder"
 			(at 142.24 187.452 90)
 			(effects
@@
 			)
 		)
-		(property "Footprint" "Capacitor_SMD:C_0402_1005Metric_Pad0.74x0.62mm_HandSolder"
+		(property "Footprint" "Capacitor_SMD:C_0805_2012Metric_Pad1.18x1.45mm_HandSolder"
 			(at 192.7352 27.94 0)
 			(effects
@@
 			)
 		)
-		(property "Footprint" "Capacitor_SMD:C_0402_1005Metric_Pad0.74x0.62mm_HandSolder"
+		(property "Footprint" "Capacitor_SMD:C_0805_2012Metric_Pad1.18x1.45mm_HandSolder"
 			(at 106.68 154.6352 0)
 			(effects
@@
 			)
 		)
-		(property "Footprint" "Capacitor_SMD:C_0402_1005Metric_Pad0.74x0.62mm_HandSolder"
+		(property "Footprint" "Capacitor_SMD:C_0805_2012Metric_Pad1.18x1.45mm_HandSolder"
 			(at 261.62 21.2852 0)
 			(effects
@@
 			)
 		)
-		(property "Footprint" "Capacitor_SMD:C_1206_3216Metric_Pad1.33x1.80mm_HandSolder"
+		(property "Footprint" "Capacitor_SMD:C_0805_2012Metric_Pad1.18x1.45mm_HandSolder"
 			(at 41.6052 182.88 0)
 			(effects
@@
 			)
 		)
-		(property "Footprint" "RF_Module:ESP32-S2-MINI-1"
+		(property "Footprint" "Espressif:ESP32-S2-SOLO"
 			(at 228.6 133.35 0)
 			(effects
@@
 			)
 		)
-		(property "Footprint" "Resistor_SMD:R_0402_1005Metric_Pad0.72x0.64mm_HandSolder"
+		(property "Footprint" "Resistor_SMD:R_0805_2012Metric_Pad1.20x1.40mm_HandSolder"
 			(at 140.208 185.42 90)
 			(effects
@@
 			)
 		)
-		(property "Footprint" "Capacitor_SMD:C_0402_1005Metric_Pad0.74x0.62mm_HandSolder"
+		(property "Footprint" "Capacitor_SMD:C_0805_2012Metric_Pad1.18x1.45mm_HandSolder"
 			(at 183.8452 146.05 0)
 			(effects
@@
 			)
 		)
-		(property "Footprint" "Resistor_SMD:R_0402_1005Metric_Pad0.72x0.64mm_HandSolder"
+		(property "Footprint" "Resistor_SMD:R_0805_2012Metric_Pad1.20x1.40mm_HandSolder"
 			(at 255.778 158.75 90)
 			(effects
@@
 			)
 		)
-		(property "Footprint" "Capacitor_SMD:C_0603_1608Metric_Pad1.08x0.95mm_HandSolder"
+		(property "Footprint" "Capacitor_SMD:C_0805_2012Metric_Pad1.18x1.45mm_HandSolder"
 			(at 45.72 153.3652 0)
 			(effects
@@
 			)
 		)
-		(property "Footprint" "Resistor_SMD:R_0402_1005Metric_Pad0.72x0.64mm_HandSolder"
+		(property "Footprint" "Resistor_SMD:R_0805_2012Metric_Pad1.20x1.40mm_HandSolder"
 			(at 207.01 31.242 90)
 			(effects
@@
 			)
 		)
-		(property "Footprint" "Capacitor_SMD:C_0402_1005Metric_Pad0.74x0.62mm_HandSolder"
+		(property "Footprint" "Capacitor_SMD:C_0805_2012Metric_Pad1.18x1.45mm_HandSolder"
 			(at 31.75 155.9052 0)
 			(effects
@@
 			)
 		)
-		(property "Footprint" "Capacitor_SMD:C_0603_1608Metric_Pad1.08x0.95mm_HandSolder"
+		(property "Footprint" "Capacitor_SMD:C_0805_2012Metric_Pad1.18x1.45mm_HandSolder"
 			(at 120.65 152.0952 0)
 			(effects
@@
 			)
 		)
-		(property "Footprint" "Capacitor_SMD:C_0201_0603Metric_Pad0.64x0.40mm_HandSolder"
+		(property "Footprint" "Capacitor_SMD:C_0805_2012Metric_Pad1.18x1.45mm_HandSolder"
 			(at 110.1852 101.6 0)
 			(effects
@@
 			)
 		)
-		(property "Footprint" "Capacitor_SMD:C_0402_1005Metric_Pad0.74x0.62mm_HandSolder"
+		(property "Footprint" "Capacitor_SMD:C_0805_2012Metric_Pad1.18x1.45mm_HandSolder"
 			(at 242.2652 31.75 0)
 			(effects
@@
 			)
 		)
-		(property "Footprint" "Resistor_SMD:R_0402_1005Metric_Pad0.72x0.64mm_HandSolder"
+		(property "Footprint" "Resistor_SMD:R_0805_2012Metric_Pad1.20x1.40mm_HandSolder"
 			(at 259.842 158.75 90)
 			(effects
@@
 			)
 		)
-		(property "Footprint" "Button_Switch_SMD:SW_Push_SPST_NO_Alps_SKRK"
+		(property "Footprint" "Connector_USB:USB_C_Receptacle_HRO_TYPE-C-31-M-12"
 			(at 251.46 140.97 0)
 			(effects

Commit message: updated schematic
Parts:
- added J9: Conn_01x02_Pin, Connector_PinHeader_1.27mm:PinHeader_1x02_P1.27mm_Vertical, symbol Connector:Conn_01x02_Pin
- J2, J3, J4, J8: footprint Connector_PinHeader_1.27mm:PinHeader_1x16_P1.27mm_Horizontal -> Connector_PinHeader_1.27mm:PinHeader_1x16_P1.27mm_Vertical
- J5: footprint Connector_PinHeader_1.27mm:PinHeader_1x02_P1.27mm_Horizontal -> Connector_PinHeader_1.27mm:PinHeader_1x02_P1.27mm_Vertical
- J6, J7: footprint Connector_PinHeader_1.27mm:PinHeader_1x04_P1.27mm_Horizontal -> Connector_PinHeader_1.27mm:PinHeader_1x04_P1.27mm_Vertical
Connections:
- net +12V: now also J9.1 (Pin_1)
- net GND: now also J9.2 (Pin_2)
Other:
- moved on the sheet: C10, C11, C12, C13, C14, C15, C18, C19, C20, C21, C22, C23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

Commit message: bet
Parts:
- J2, J3, J4, J8: footprint Connector_PinHeader_1.27mm:PinHeader_1x16_P1.27mm_Vertical -> Connector_PinHeader_2.54mm:PinHeader_1x16_P2.54mm_Vertical
- J5, J9: footprint Connector_PinHeader_1.27mm:PinHeader_1x02_P1.27mm_Vertical -> Connector_PinHeader_2.54mm:PinHeader_1x02_P2.54mm_Vertical
- J6, J7: footprint Connector_PinHeader_1.27mm:PinHeader_1x04_P1.27mm_Vertical -> Connector_PinHeader_2.54mm:PinHeader_1x04_P2.54mm_Vertical
Changed lines of the file:
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@@
 			)
 		)
-		(property "Footprint" "Connector_PinHeader_1.27mm:PinHeader_1x16_P1.27mm_Vertical"
+		(property "Footprint" "Connector_PinHeader_2.54mm:PinHeader_1x16_P2.54mm_Vertical"
 			(at 176.53 48.26 0)
 			(effects
@@
 			)
 		)
-		(property "Footprint" "Connector_PinHeader_1.27mm:PinHeader_1x16_P1.27mm_Vertical"
+		(property "Footprint" "Connector_PinHeader_2.54mm:PinHeader_1x16_P2.54mm_Vertical"
 			(at 134.62 48.26 0)
 			(effects
@@
 			)
 		)
-		(property "Footprint" "Connector_PinHeader_1.27mm:PinHeader_1x16_P1.27mm_Vertical"
+		(property "Footprint" "Connector_PinHeader_2.54mm:PinHeader_1x16_P2.54mm_Vertical"
 			(at 92.71 46.99 0)
 			(effects
@@
 			)
 		)
-		(property "Footprint" "Connector_PinHeader_1.27mm:PinHeader_1x16_P1.27mm_Vertical"
+		(property "Footprint" "Connector_PinHeader_2.54mm:PinHeader_1x16_P2.54mm_Vertical"
 			(at 50.8 46.99 0)
 			(effects
@@
 			)
 		)
-		(property "Footprint" "Connector_PinHeader_1.27mm:PinHeader_1x04_P1.27mm_Vertical"
+		(property "Footprint" "Connector_PinHeader_2.54mm:PinHeader_1x04_P2.54mm_Vertical"
 			(at 82.55 114.3 0)
 			(effects
@@
 			)
 		)
-		(property "Footprint" "Connector_PinHeader_1.27mm:PinHeader_1x02_P1.27mm_Vertical"
+		(property "Footprint" "Connector_PinHeader_2.54mm:PinHeader_1x02_P2.54mm_Vertical"
 			(at 143.51 168.91 0)
 			(effects
@@
 			)
 		)
-		(property "Footprint" "Connector_PinHeader_1.27mm:PinHeader_1x02_P1.27mm_Vertical"
+		(property "Footprint" "Connector_PinHeader_2.54mm:PinHeader_1x02_P2.54mm_Vertical"
 			(at 24.13 176.53 0)
 			(effects
@@
 			)
 		)
-		(property "Footprint" "Connector_PinHeader_1.27mm:PinHeader_1x04_P1.27mm_Vertical"
+		(property "Footprint" "Connector_PinHeader_2.54mm:PinHeader_1x04_P2.54mm_Vertical"
 			(at 157.48 115.57 0)
 			(effects

Commit message: Test points added
Parts:
- added TP1, TP2, TP3, TP4, TP5, TP6, TP7: TestPoint, symbol Connector:TestPoint
Connections:
- net +12V: now also TP1.1, TP6.1, TP7.1
- net +3.3V: now also TP5.1
- net +5V: now also TP2.1, TP3.1
- net GND: now also TP4.1

Commit message: TestPoints named and layouts 1.5x1.5
Parts:
- TP1: value TestPoint -> PowerSupply_TestPoint; footprint (none) -> TestPoint:TestPoint_Pad_1.5x1.5mm
- TP2: value TestPoint -> 12VConverter_TestPoint; footprint (none) -> TestPoint:TestPoint_Pad_1.5x1.5mm
- TP3: value TestPoint -> BeforeEM_TestPoint; footprint (none) -> TestPoint:TestPoint_Pad_1.5x1.5mm
- TP4: value TestPoint -> AfterEM_TestPoint; footprint (none) -> TestPoint:TestPoint_Pad_1.5x1.5mm
- TP5: value TestPoint -> 3.3VConverter_TestPoint; footprint (none) -> TestPoint:TestPoint_Pad_1.5x1.5mm
- TP6: value TestPoint -> TMC_Input1_TestPoint; footprint (none) -> TestPoint:TestPoint_Pad_1.5x1.5mm
- TP7: value TestPoint -> TMC_Input2_TestPoint; footprint (none) -> TestPoint:TestPoint_Pad_1.5x1.5mm
Changed lines of the file:
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@@
 			)
 		)
-		(property "Value" "TestPoint"
+		(property "Value" "12VConverter_TestPoint"
 			(at 118.11 175.7679 0)
 			(effects
@@
 			)
 		)
-		(property "Footprint" ""
+		(property "Footprint" "TestPoint:TestPoint_Pad_1.5x1.5mm"
 			(at 120.65 177.8 0)
 			(effects
@@
 			)
 		)
-		(property "Value" "TestPoint"
+		(property "Value" "BeforeEM_TestPoint"
 			(at 138.43 178.5619 0)
 			(effects
@@
 			)
 		)
-		(property "Footprint" ""
+		(property "Footprint" "TestPoint:TestPoint_Pad_1.5x1.5mm"
 			(at 130.81 173.99 0)
 			(effects
@@
 			)
 		)
-		(property "Value" "TestPoint"
+		(property "Value" "AfterEM_TestPoint"
 			(at 163.83 171.9579 0)
 			(effects
@@
 			)
 		)
-		(property "Footprint" ""
+		(property "Footprint" "TestPoint:TestPoint_Pad_1.5x1.5mm"
 			(at 166.37 173.99 0)
 			(effects
@@
 			)
 		)
-		(property "Value" "TestPoint"
+		(property "Value" "TMC_Input1_TestPoint"
 			(at 132.08 145.2879 0)
 			(effects
@@
 			)
 		)
-		(property "Footprint" ""
+		(property "Footprint" "TestPoint:TestPoint_Pad_1.5x1.5mm"
 			(at 134.62 147.32 0)
 			(effects
@@
 			)
 		)
-		(property "Value" "TestPoint"
+		(property "Value" "3.3VConverter_TestPoint"
 			(at 220.98 139.6999 90)
 			(effects
@@
 			)
 		)
-		(property "Footprint" ""
+		(property "Footprint" "TestPoint:TestPoint_Pad_1.5x1.5mm"
 			(at 215.9 143.51 0)
 			(effects
@@
 			)
 		)
-		(property "Value" "TestPoint"
+		(property "Value" "TMC_Input2_TestPoint"
 			(at 57.15 146.5579 0)
 			(effects
@@
 			)
 		)
-		(property "Footprint" ""
+		(property "Footprint" "TestPoint:TestPoint_Pad_1.5x1.5mm"
 			(at 59.69 148.59 0)
 			(effects
@@
 			)
 		)
-		(property "Value" "TestPoint"
+		(property "Value" "PowerSupply_TestPoint"
 			(at 36.83 174.4979 0)
 			(effects
@@
 			)
 		)
-		(property "Footprint" ""
+		(property "Footprint" "TestPoint:TestPoint_Pad_1.5x1.5mm"
 			(at 39.37 176.53 0)
 			(effects
