File: kicad/Motherboard/Motherboard.kicad_sch (KiCad schematic)
At the start: 71 parts, among them J1 USB_C_Receptacle_USB2.0, J10 Conn_01x08_Pin, J11 Conn_01x08_Pin, J12 Conn_01x08_Pin, J13 Conn_01x08_Pin, J2 Conn_01x02_Pin, J3 Conn_01x04_Pin, J4 Conn_01x04_Pin, J5 Conn_01x02_Pin, J6 Conn_01x08_Pin, J7 Conn_01x08_Pin, J8 Conn_01x08_Pin, J9 Conn_01x08_Pin, Q1 DMN3404L, SW1 Reset, SW2 Boot, U1 ESP32-S2-SOLO, U2 LD1117S33TR_SOT223, U3 TCA9535RTWR, U4 TCA9535RTWR, U5 TCA9535RTWR, U6 TCA9535RTWR, U7 TMC2208-LA, U8 TMC2208-LA, U9 LM2575-5.0BT

Commit message: finish pls sia
Parts:
- added D5: 1N5819, Diode_THT:D_DO-41_SOD81_P5.08mm_Vertical_AnodeUp, symbol Device:D_Schottky
- U7, U8: value TMC2208-LA -> TMC2209-LA
Connections:
- net +12V: now also D5.1 (K); no longer F1.2
- new net: D5.2 (A), F1.2
Changed lines of the file:
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@@
 	(wire
 		(pts
-			(xy 38.1 179.07) (xy 43.18 179.07)
-		)
-		(stroke
-			(width 0)
-			(type default)
-		)
-	)
-	(wire
-		(pts
 			(xy 46.99 152.4) (xy 46.99 157.48)
 		)
@@
 			)
 		)
-		(property "Value" "TMC2208-LA"
+		(property "Value" "TMC2209-LA"
 			(at 146.05 134.366 0)
 			(effects
@@
 	(symbol
 		(lib_id "power:+12V")
-		(at 43.18 179.07 0)
+		(at 45.72 179.07 0)
 		(unit 1)
 		(exclude_from_sim no)
@@
 		(dnp no)
 		(property "Reference" "#PWR034"
-			(at 43.18 182.88 0)
+			(at 45.72 182.88 0)
 			(effects
 				(font
@@
 		)
 		(property "Value" "+12V"
-			(at 46.482 177.292 0)
+			(at 49.022 177.292 0)
 			(effects
 				(font
@@
 		)
 		(property "Footprint" ""
-			(at 43.18 179.07 0)
+			(at 45.72 179.07 0)
 			(effects
 				(font
@@
 		)
 		(property "Datasheet" ""
-			(at 43.18 179.07 0)
+			(at 45.72 179.07 0)
 			(effects
 				(font
@@
 		)
 		(property "Description" "Power symbol creates a global label with name \"+12V\""
-			(at 43.18 179.07 0)
+			(at 45.72 179.07 0)
 			(effects
 				(font
@@
 		)
 		(property "Value" "Polyfuse"
-			(at 34.544 176.276 90)
+			(at 34.29 176.53 90)
 			(effects
 				(font
@@
 			)
 		)
-		(property "Value" "TMC2208-LA"
+		(property "Value" "TMC2209-LA"
 			(at 88.9 134.366 0)
 			(effects
@@
 					(unit 1)
 				)
+			)
+		)
+	)
+	(symbol
+		(lib_id "Device:D_Schottky")
+		(at 41.91 179.07 180)
+		(unit 1)
+		(exclude_from_sim no)
+		(in_bom yes)
+		(on_board yes)
+		(dnp no)
+		(property "Reference" "D5"
+			(at 41.91 176.53 0)
+			(effects
+				(font
+					(size 1.27 1.27)
+				)
+				(justify right)
+			)
+		)
+		(property "Value" "1N5819"
+			(at 38.354 181.61 0)
+			(effects
+				(font
+					(size 1.27 1.27)
+				)
+				(justify right)
+			)
+		)
+		(property "Footprint" "Diode_THT:D_DO-41_SOD81_P5.08mm_Vertical_AnodeUp"
+			(at 41.91 179.07 0)
+			(effects
+				(font
+					(size 1.27 1.27)
+				)
+				(hide yes)
+			)
+		)
+		(property "Datasheet" "~"
+			(at 41.91 179.07 0)
+			(effects
+				(font
+					(size 1.27 1.27)
+				)
+				(hide yes)
+			)
+		)
+		(property "Description" "Schottky diode"
+			(at 41.91 179.07 0)
+			(effects
+				(font
+					(size 1.27 1.27)
+				)
+				(hide yes)
+			)
+		)
+		(pin "2"
+		)
+		(pin "1"
+		)
+		(instances
+			(project "Motherboard"
+				(path "/6e7606c8-26d5-4d26-b509-210c4758a44d"
+					(reference "D5")
+					(unit 1)
+				)
