File: kicad/Motherboard/_autosave-Motherboard.kicad_pcb (KiCad board)
At the start: 2 copper layers, 57.3 x 62.8 mm, 84 parts, among them J1 USB_C_Receptacle_USB2.0, J10 Conn_01x08_Pin, J11 Conn_01x08_Pin, J12 Conn_01x08_Pin, J13 Conn_01x08_Pin, J2 Conn_01x02_Pin, J3 Conn_01x04_Pin, J4 Conn_01x04_Pin, J5 Conn_01x02_Pin, J6 Conn_01x08_Pin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

Commit message: bruh
Parts:
- removed TP2: 12VConverter_TestPoint, TestPoint:TestPoint_Pad_1.5x1.5mm
- moved TP3 21.5 mm to (132.9, 73.3)
- moved D2 6.24 mm to (164.0, 85.2), turned to 180 degrees
- moved R10 5.69 mm to (139.9, 89.3)
- moved D1 5.13 mm to (164.1, 81.5)
- moved R2 4.73 mm to (136.4, 91.4), turned to -90 degrees
- moved C3 3.83 mm to (164.6, 73.7)
- moved C8 3.62 mm to (160.4, 92.5)
- moved C7 3.50 mm to (161.1, 73.7), turned to -90 degrees
- moved C5 3.40 mm to (139.8, 92.8)
- moved C1 3.08 mm to (151.2, 89.9)
- moved SW2 2.67 mm to (144.0, 91.0), turned to 90 degrees
- moved SW1 2.50 mm to (147.9, 91.0)
- moved L1 2.44 mm to (154.1, 90.5)
- moved D4 1.78 mm to (164.0, 89.0)
- moved TP1 1.31 mm to (165.9, 92.6)
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Routing:
- net Net-(U1-EN): track 42.4 -> 17.1 mm
- net Net-(U1-GPIO0): track 19.2 -> 3.27 mm
- net SDA: track 16.1 -> 0.34 mm, vias 2 -> 1
- net ENN_2: track 13.9 -> 0.00 mm, vias 1 -> 0
- net +5V: track 65.3 -> 54.4 mm, vias 1 -> 0
- net Net-(D1-K): track 39.1 -> 49.6 mm
- net Net-(D5-A): track 22.7 -> 30.6 mm, vias 0 -> 1
- net Net-(J5-Pin_1): track 17.3 -> 10.5 mm
- net Net-(D2-A): track 9.46 -> 16.2 mm
- net SCL: track 17.4 -> 12.8 mm, vias 2 -> 0
- net MAGCT: track 5.37 -> 2.20 mm
- net STEP_2: track 2.85 -> 0.00 mm, vias 2 -> 0
- net VS_1: track 76.6 -> 79.0 mm, vias 6 -> 7
- net Net-(Q1-G): track 16.8 -> 15.3 mm
- net +3.3V: track 52.4 -> 53.6 mm
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Other:
- board text added: "U1"
